File: cam_pcb/cam_pcb.kicad_pcb (KiCad board)
At the start: 2 copper layers, 50 x 40 mm, 33 parts, among them J1 TYPE-C-31-M-12, J2 Conn_01x24, U1 W25Q128JVS, U2 RP2040, U3 NCP1117-3.3_SOT223, X1 12Mhz

Commit message: all but camera
Parts:
- removed R2: DNF, Resistor_SMD:R_0402_1005Metric
- moved U3 26.5 mm to (132.1, 116.2)
- moved C17 23.8 mm to (133.2, 120.8), turned to 180 degrees
- moved J2 5.83 mm to (145.8, 116.3), turned to 180 degrees
Routing:
- net +3V3: track 39.2 -> 52.7 mm
- net VBUS: track 10.0 -> 19.2 mm
- net GND: track 43.5 -> 46.6 mm, vias 21 -> 22
- added copper zone on F.Cu, net +3V3
- added copper zone on B.Cu, net GND
- removed copper zone on F.Cu, net GND
