File: cam_pcb/cam_pcb.kicad_sch (KiCad schematic)
At the start: 33 parts, among them J1 TYPE-C-31-M-12, J2 Conn_01x24, U1 W25Q128JVS, U2 RP2040, U3 NCP1117-3.3_SOT223, X1 12Mhz

Commit message: all but camera
Other:
- note added: "Minor adjustments need to be made here. https://cdn.sparkfun.com/assets/7/f/c/8/3/HM01B0-MNA-Datasheet.pdf"
Changed lines of the file:
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@@
 		)
 	)
+	(text "Minor adjustments need to be made here.\nhttps://cdn.sparkfun.com/assets/7/f/c/8/3/HM01B0-MNA-Datasheet.pdf"
+		(exclude_from_sim no)
+		(at 155.194 117.602 90)
+		(effects
+			(font
+				(size 1 1)
+			)
+		)
+	)
 	(text "RP2040 Cam PCB 1"
 		(exclude_from_sim no)
@@
 		(on_board yes)
 		(dnp no)
-		(fields_autoplaced yes)
 		(property "Reference" "J2"
-			(at 153.67 114.2999 0)
+			(at 163.83 111.506 0)
 			(effects
 				(font
@@
 		)
 		(property "Value" "Conn_01x24"
-			(at 153.67 116.8399 0)
+			(at 158.242 114.554 0)
 			(effects
 				(font
